Commit message: Implementacao do trabalho 2

File: description/r2d2.urdf.xacro (robot description, xacro)
@@ -4,5 +4,7 @@
   <xacro:property name="cylinder_radius" value="0.1"/>
   <xacro:property name="cylinder_length" value="0.3"/>
-  <xacro:property name="box_size" value="0.33 0.05 0.03"/>
+  <xacro:property name="base_length" value="0.33"/>
+  <xacro:property name="base_width"  value="0.05"/>
+  <xacro:property name="base_height" value="0.03"/>
   <xacro:property name="sphere_radius" value="0.1"/>
   <xacro:property name="wheel_radius" value="0.06"/>
@@ -18,4 +20,25 @@
     <color rgba="0 0 0 1"/>
   </material>
+  <!-- Definição de algumas propriedades inerciais -->
+  <xacro:macro name="box_inertia" params="m w h d">
+    <inertial>
+      <origin xyz="0 0 0" rpy="${pi/2} 0 ${pi/2}"/>
+      <mass value="${m}"/>
+      <inertia ixx="${(m/12) * (h*h + d*d)}" ixy="0.0" ixz="0.0" iyy="${(m/12) * (w*w + d*d)}" iyz="0.0" izz="${(m/12) * (w*w + h*h)}"/>
+    </inertial>
+  </xacro:macro>
+  <xacro:macro name="cylinder_inertia" params="m r h">
+    <inertial>
+      <origin xyz="0 0 0" rpy="${pi/2} 0 0" />
+      <mass value="${m}"/>
+      <inertia ixx="${(m/12) * (3*r*r + h*h)}" ixy = "0" ixz = "0" iyy="${(m/12) * (3*r*r + h*h)}" iyz = "0" izz="${(m/2) * (r*r)}"/>
+    </inertial>
+  </xacro:macro>
+  <xacro:macro name="sphere_inertia" params="m r">
+    <inertial>
+      <mass value="${m}"/>
+      <inertia ixx="${(2/5) * m * (r*r)}" ixy="0.0" ixz="0.0" iyy="${(2/5) * m * (r*r)}" iyz="0.0" izz="${(2/5) * m * (r*r)}"/>
+    </inertial>
+  </xacro:macro>
   <!-- Link base -->
   <link name="base_link">
@@ -33,8 +56,5 @@
       <origin xyz="0 0 0" rpy="0.5 0 0"/>
     </collision>
-    <inertial>
-      <mass value="10"/>
-      <inertia ixx="1.0" ixy="0.0" ixz="0.0" iyy="1.0" iyz="0.0" izz="1.0"/>
-    </inertial>
+    <xacro:cylinder_inertia m="10" r="${cylinder_radius}" h="${cylinder_length}"/>
   </link>
   <!-- Função para criar pernas -->
@@ -43,5 +63,5 @@
       <visual>
         <geometry>
-          <box size="${box_size}"/>
+          <box size="${base_length} ${base_width} ${base_height}"/>
         </geometry>
         <origin xyz="0 0 0" rpy="0 1.58 0"/>
@@ -50,12 +70,9 @@
       <collision>
         <geometry>
-          <box size="${box_size}"/>
+          <box size="${base_length} ${base_width} ${base_height}"/>
         </geometry>
           <origin xyz="0 0 0" rpy="0 1.58 0"/>
       </collision>
-      <inertial>
-        <mass value="10"/>
-        <inertia ixx="0.01" ixy="0.0" ixz="0.0" iyy="0.01" iyz="0.0" izz="0.01"/>
-      </inertial>
+      <xacro:box_inertia m="1" w="${base_width}" d="${base_length}" h="${base_height}"/>
     </link>
     <joint name="base_to_${name}" type="fixed">
@@ -82,8 +99,5 @@
       <origin xyz="0.0 0.0 0.01" rpy="0 0 0"/>
     </collision>
-    <inertial>
-      <mass value="2"/>
-      <inertia ixx="0.01" ixy="0.0" ixz="0.0" iyy="0.01" iyz="0.0" izz="0.01"/>
-    </inertial>
+    <xacro:sphere_inertia m="2" r="${sphere_radius}"/>
   </link>
   <joint name="base_to_head" type="fixed">
@@ -108,8 +122,5 @@
       <origin xyz="0 0 0" rpy="0.5 0 0"/>
     </collision>
-    <inertial>
-      <mass value="10"/>
-      <inertia ixx="0.01" ixy="0.0" ixz="0.0" iyy="0.01" iyz="0.0" izz="0.01"/>
-    </inertial>
+    <xacro:box_inertia m="10" w="0.1" h="0.1" d="0.06"/>
   </link>
   <joint name="base_to_base_bottom" type="fixed">
@@ -134,8 +145,5 @@
         </geometry>
       </collision>
-      <inertial>
-        <mass value="2.5"/>
-        <inertia ixx="0.01" ixy="0.0" ixz="0.0" iyy="0.01" iyz="0.0" izz="0.01"/>
-      </inertial>
+      <xacro:cylinder_inertia m="2.5" r="${wheel_radius}" h="${wheel_length}"/>
     </link>
     <joint name="${parent_link}_to_${name}" type="${type}">
@@ -151,4 +159,112 @@
   <xacro:wheel name="wheel_back_right" parent_link="base_link" pos="0.15 -0.05 -0.2" type = "continuous"/>
   <xacro:wheel name="wheel_back_left" parent_link="base_link" pos="-0.15 -0.05 -0.2" type = "continuous"/>
+  <!-- Garra -->
+  <link name="gripper_pole">
+    <visual>
+      <geometry>
+        <cylinder length="0.2" radius="0.01"/>
+      </geometry>
+      <origin rpy="0 0 0" xyz="0 0 -0.1"/>
+      <material name="blue"/>
+    </visual>
+    <collision>
+      <geometry>
+        <cylinder length="0.2" radius="0.01"/>
+      </geometry>
+      <origin rpy="0 0 0" xyz="0 0 -0.1"/>
+    </collision>
+    <xacro:cylinder_inertia m="0.01" r="0.01" h="0.2"/>
+  </link>
+  <joint name="gripper_extension" type="revolute">
+    <axis xyz="-1 0 0"/>
+    <limit effort="50.0" lower="-1.57075" upper="0.35" velocity="0.5"/>
+    <origin rpy="${pi/2} 0 0" xyz="0 0.01 0.15"/>
+    <parent link="base_link"/>
+    <child link="gripper_pole"/>
+  </joint>
+  <link name="left_gripper">
+    <visual>
+      <geometry>
+        <box size="0.1 0.02 0.02"/> <!-- Comprimento, largura, altura -->
+      </geometry>
+      <origin rpy="0 0 0" xyz="0 0 0"/>
+      <material name="black"/>
+    </visual>
+    <collision>
+      <geometry>
+        <box size="0.1 0.02 0.02"/>
+      </geometry>
+    </collision>
+    <xacro:box_inertia m="0.015" w="0.02" h="0.02" d="0.1"/>
+  </link>
+  <joint name="left_gripper_joint" type="prismatic">
+    <axis xyz="0 0 1"/>
+    <limit effort="100.0" lower="-0.1" upper="0" velocity="0.25"/>
+    <origin xyz="-0.01 0 -0.23" rpy="0 ${pi/2} 0"/>
+    <parent link="gripper_pole"/>
+    <child link="left_gripper"/>
+  </joint>
+  <joint name="left_tip_joint" type="fixed">
+    <origin rpy="0 -0.2 0" xyz="0.08 0 0"/>
+    <parent link="left_gripper"/>
+    <child link="left_tip"/>
+  </joint>
+  <link name="left_tip">
+    <visual>
+      <geometry>
+        <box size="0.06 0.01 0.01"/>
+      </geometry>
+      <origin rpy="0 0 0" xyz="0 0 0"/>
+      <material name="white"/>
+    </visual>
+    <collision>
+      <geometry>
+        <box size="0.06 0.01 0.01"/>
+      </geometry>
+    </collision>
+    <xacro:box_inertia m="0.005" w="0.01" h="0.01" d="0.06"/>
+  </link>
+  <link name="right_gripper">
+    <visual>
+      <geometry>
+        <box size="0.1 0.02 0.02"/>
+      </geometry>
+      <origin rpy="0 0 0" xyz="0 0 0"/>
+      <material name="black"/>
+    </visual>
+    <collision>
+      <geometry>
+        <box size="0.1 0.02 0.02"/>
+      </geometry>
+    </collision>
+    <xacro:box_inertia m="0.015" w="0.02" h="0.02" d="0.1"/>
+  </link>
+  <joint name="right_gripper_joint" type="prismatic">
+    <axis xyz="0 0 1"/>
+    <limit effort="100.0" lower="0" upper="0.1" velocity="0.25"/>
+    <origin rpy="0 ${pi/2} 0" xyz="0.01 0 -0.23"/>
+    <parent link="gripper_pole"/>
+    <child link="right_gripper"/>
+  </joint>
+  <link name="right_tip">
+    <visual>
+      <origin rpy="0 0 0" xyz="0 0 0"/>
+      <geometry>
+        <box size="0.06 0.01 0.01"/>
+      </geometry>
+      <material name="white"/>
+    </visual>
+    <collision>
+      <geometry>
+        <box size="0.06 0.01 0.01"/>
+      </geometry>
+    </collision>
+    <xacro:box_inertia m="0.005" w="0.01" h="0.01" d="0.06"/>
+  </link>
+  <joint name="right_tip_joint" type="fixed">
+    <origin rpy="0 0.2 0" xyz="0.08 0 0"/>
+    <parent link="right_gripper"/>
+    <child link="right_tip"/>
+  </joint>
 <!-- End Robot -->
 <!-- IMU -->
@@ -161,5 +277,5 @@
   <collision>
     <geometry>
-      <box size="0.1 0.1 0.1"/>
+      <box size="0.05 0.05 0.05"/>
     </geometry>
   </collision>
@@ -246,16 +362,11 @@
     <plugin>ign_ros2_control/IgnitionSystem</plugin>
   </hardware>
-  <!-- Definição do primeiro atuador, correspondente à roda dereita traseira -->
+  <!-- Definição das rodas -->
   <joint name="base_link_to_wheel_back_right">
-    <!-- Interface de comando de velocidade angular (por exemplo, rad/s) para essa junta -->
     <command_interface name="velocity">
-      <!-- Valor mínimo permitido para o comando de velocidade (limite inferior) -->
       <param name="min">-1</param>
-      <!-- Valor máximo permitido para o comando de velocidade (limite superior) -->
       <param name="max">1</param>
     </command_interface>
-    <!-- Interface de estado que fornece a posição atual da junta (por exemplo, em radianos) -->
     <state_interface name="position"/>
-    <!-- Interface de estado que fornece a velocidade atual da junta (por exemplo, em rad/s) -->
     <state_interface name="velocity"/>
   </joint>
@@ -284,8 +395,32 @@
     <state_interface name="velocity"/>
   </joint>
+    <joint name="gripper_extension">
+      <command_interface name="position">
+        <param name="min">-1.57075</param>
+        <param name="max">0.2</param>
+      </command_interface>
+      <state_interface name="position"/>
+      <state_interface name="velocity"/>
+    </joint>
+    <joint name="left_gripper_joint">
+      <command_interface name="position">
+        <param name="min">0.0</param>
+        <param name="max">0.1</param>
+      </command_interface>
+      <state_interface name="position"/>
+      <state_interface name="velocity"/>
+    </joint>
+    <joint name="right_gripper_joint">
+      <command_interface name="position">
+        <param name="min">-0.1</param>
+        <param name="max">0.0</param>
+      </command_interface>
+      <state_interface name="position"/>
+      <state_interface name="velocity"/>
+    </joint>
 </ros2_control>
   <gazebo>
     <plugin filename="ign_ros2_control-system" name="ign_ros2_control::IgnitionROS2ControlPlugin">
-      <parameters>$(find prm)/config/diff_drive_controller_velocity.yaml</parameters>
+      <parameters>$(find prm)/config/controller_config.yaml</parameters>
     </plugin>
   </gazebo>
@@ -371,22 +506,22 @@
 </joint>
 <gazebo reference="camera_link">
-  <sensor name="robot_cam" type="camera">
-   <camera>
-      <horizontal_fov>1.047</horizontal_fov>
-      <image>
-        <width>320</width>
-        <height>240</height>
-      </image>
-      <clip>
-        <near>0.1</near>
-        <far>100</far>
-      </clip>
-    </camera>
-    <always_on>1</always_on>
-    <update_rate>30</update_rate>
-    <visualize>true</visualize>
-    <topic>robot_cam</topic>
-    <enable_metrics>true</enable_metrics>
-  </sensor>
+    <sensor name="robot_cam" type="segmentation">
+      <topic>robot_cam</topic>
+      <camera>
+        <segmentation_type>semantic</segmentation_type>
+        <horizontal_fov>1.57</horizontal_fov>
+        <image>
+          <width>320</width>
+          <height>240</height>
+        </image>
+        <clip>
+          <near>0.1</near>
+          <far>100</far>
+        </clip>
+      </camera>
+      <always_on>1</always_on>
+      <update_rate>15</update_rate>
+      <visualize>true</visualize>
+    </sensor>
 </gazebo>
   <gazebo>

Commit message: Update gripper extension joint limit for improved functionality; adjust collection distance constant for better obstacle handling.

File: description/r2d2.urdf.xacro (robot description, xacro)
@@ -178,5 +178,5 @@
   <joint name="gripper_extension" type="revolute">
     <axis xyz="-1 0 0"/>
-    <limit effort="50.0" lower="-1.57075" upper="0.35" velocity="0.5"/>
+    <limit effort="50.0" lower="-1.57075" upper="0.5" velocity="0.5"/>
     <origin rpy="${pi/2} 0 0" xyz="0 0.01 0.15"/>
     <parent link="base_link"/>
